File: Hardware/PiWeatherShield/PiWeatherShield.kicad_sch (KiCad schematic)
At the start: 11 parts, among them U1 Raspberry Pi inner pin row, U2 SSD1306DisplayBoard, U3 Si7021Board, U4 BME280Board

Commit message: init version
Parts:
- removed C1: 2u2, symbol Device:C_Polarized_Small
- removed C2, C3, C4, C5: 100n, symbol Device:C
- removed R1: TBD, symbol Device:R
- removed U1: Raspberry Pi inner pin row, symbol PiWeatherShieldSymbolLibrary:RaspberryInnerPinHeader
- removed U3: Si7021Board, symbol PiWeatherShieldSymbolLibrary:Si7021Board
- added C6, C7, C8, C9: 100n, Capacitor_SMD:C_0805_2012Metric, symbol Device:C
- added J1: Conn_02x20_Odd_Even, Connector_PinSocket_2.54mm:PinSocket_2x20_P2.54mm_Horizontal, symbol Connector_Generic:Conn_02x20_Odd_Even
- added J2: Conn_02x20_Odd_Even, Connector_PinHeader_2.54mm:PinHeader_2x20_P2.54mm_Horizontal, symbol Connector_Generic:Conn_02x20_Odd_Even
- added R3: 2k2, Resistor_SMD:R_0805_2012Metric, symbol Device:R
- added TP1, TP2, TP3, TP4: TestPoint, TestPoint:TestPoint_Pad_D2.0mm, symbol Connector:TestPoint
- added U1: Si7021Board, PiWeatherShield:SIP-4, symbol PiWeatherShieldSymbolLibrary:Si7021Board
- added U3: GY- SGP30/SGP40, PiWeatherShield:GY- SGP30SGP40, symbol PiWeatherShieldSymbolLibrary:GY- SGP30/SGP40
- R2: value TBD -> 2k2; footprint (none) -> Resistor_SMD:R_0805_2012Metric
- U2: footprint (none) -> PiWeatherShield:SSD1306DisplayBoard
- U4: footprint (none) -> PiWeatherShield:BME280Board
Connections:
- net GND: now also U2.3 (GND), C6.2, C7.2, C8.2, C9.2, J1.14 (Pin_14), J1.20 (Pin_20), J1.25 (Pin_25), J1.30 (Pin_30), J1.34 (Pin_34), J1.39 (Pin_39), J1.6 (Pin_6), J1.9 (Pin_9), J2.14 (Pin_14), J2.20 (Pin_20), J2.25 (Pin_25), J2.30 (Pin_30), J2.34 (Pin_34), J2.39 (Pin_39), J2.6 (Pin_6), J2.9 (Pin_9), TP2.1, U1.4 (GND), U3.3 (GND); no longer U2.2 (GND)
- net GPIO2/SDA: now reaches U4.3 (SDA)
- net GPIO2/SDA: now also U2.2 (SDA), J1.3 (Pin_3), J2.3 (Pin_3), R3.2, TP3.1, U1.2 (SDA), U3.1 (SDA); no longer U2.3 (SDA)
- net GPIO3/SCL: now reaches R2.2, U4.4 (SCL)
- net GPIO3/SCL: now also U2.1 (SCL), J1.5 (Pin_5), J2.5 (Pin_5), TP4.1, U1.1 (SCL), U3.2 (SCL); no longer U2.4 (SCL)
- net VCC renamed +3.3V
- net +3.3V: now also U2.4 (VCC), C6.1, C7.1, C8.1, C9.1, J1.1 (Pin_1), J1.17 (Pin_17), J2.1 (Pin_1), J2.17 (Pin_17), R3.1, TP1.1, U1.3 (VCC), U3.4 (VCC); no longer U2.1 (VCC)
- new net 5V: J1.2 (Pin_2), J1.4 (Pin_4), J2.2 (Pin_2), J2.4 (Pin_4)
- new net GPIO0/ID_SD: J1.27 (Pin_27), J2.27 (Pin_27)
- new net GPIO1: J1.28 (Pin_28), J2.28 (Pin_28)
- new net GPIO10/MOSI: J1.19 (Pin_19), J2.19 (Pin_19)
- new net GPIO11/SCLK: J1.23 (Pin_23), J2.23 (Pin_23)
- new net GPIO12: J1.32 (Pin_32), J2.32 (Pin_32)
- new net GPIO13/PCM_FS: J1.35 (Pin_35), J2.35 (Pin_35)
- new net GPIO13/PWM1: J1.33 (Pin_33), J2.33 (Pin_33)
- new net GPIO14: J1.8 (Pin_8), J2.8 (Pin_8)
- new net GPIO15: J1.10 (Pin_10), J2.10 (Pin_10)
- new net GPIO16: J1.36 (Pin_36), J2.36 (Pin_36)
- new net GPIO17: J1.11 (Pin_11), J2.11 (Pin_11)
- new net GPIO18: J1.12 (Pin_12), J2.12 (Pin_12)
- new net GPIO20: J1.38 (Pin_38), J2.38 (Pin_38)
- new net GPIO21: J1.40 (Pin_40), J2.40 (Pin_40)
- new net GPIO22: J1.15 (Pin_15), J2.15 (Pin_15)
- new net GPIO23: J1.16 (Pin_16), J2.16 (Pin_16)
- new net GPIO24: J1.18 (Pin_18), J2.18 (Pin_18)
- new net GPIO25: J1.22 (Pin_22), J2.22 (Pin_22)
- new net GPIO26: J1.37 (Pin_37), J2.37 (Pin_37)
- new net GPIO27: J1.13 (Pin_13), J2.13 (Pin_13)
- new net GPIO4/GPCLK0: J1.7 (Pin_7), J2.7 (Pin_7)
- new net GPIO5: J1.29 (Pin_29), J2.29 (Pin_29)
- new net GPIO6: J1.31 (Pin_31), J2.31 (Pin_31)
- new net GPIO7: J1.26 (Pin_26), J2.26 (Pin_26)
- new net GPIO8: J1.24 (Pin_24), J2.24 (Pin_24)
- new net GPIO9/MISO: J1.21 (Pin_21), J2.21 (Pin_21)
- no-connect marks 14 -> 0
Other:
- moved on the sheet: R2, U2, U4
